File: Electronic_Modular/Sumo_Geral_Modular/Sumo_Geral_Modular.kicad_sch (KiCad schematic)
At the start: 50 parts, among them J1 Bateria, J10 ESC1, J11 ESC2, J12 USB_B_Micro, J13 ADSN-9500, J14 PS ADSN-9500, J15 MPU-6050, J2 VL53L0X 1, J3 VL53L0X 2, J4 VL53L0X 3, J5 VS1838B, J8 Motor A, J9 Motor B, Q1 S8050, Q2 S8050, SW2 EN, SW3 BOOT, U1 AMS1117-5.0, U2 AMS1117-3.3, U3 CH340C

Commit message: chore: Add/Update 3D models on PCB
Parts:
- 6_Pins_Button1: footprint Button_Switch_THT:Nidec_Copal_SH-7010C -> esp32_devkit_v1_doit:Push_Button_6_pins
- D1: value LED -> BLUE
- D3, D5: value LED -> RED
- H_Bridge1: footprint esp32_devkit_v1_doit:H_Bridge -> esp32_devkit_v1_doit:H_Bridge_with_headers
- J2, J3, J4: footprint Connector_JST:JST_XH_B5B-XH-AM_1x05_P2.50mm_Vertical -> Connector_JST:JST_XH_B5B-XH-A_1x05_P2.50mm_Vertical
- J8, J9: footprint Connector_JST:JST_XH_B2B-XH-AM_1x02_P2.50mm_Vertical -> Connector_JST:JST_XH_B2B-XH-A_1x02_P2.50mm_Vertical
- R13: value 1K -> 130R
- R3: value 1K -> 500R
Connections:
- net I00: no longer Q2.3 (C)
- net IO0: now also Q2.3 (C)
- net at J9.1 (Pin_1): now also H_Bridge1.7 (BO1); no longer H_Bridge1.6 (BO2)
- net at J9.2 (Pin_2): now also H_Bridge1.6 (BO2); no longer H_Bridge1.7 (BO1)
- no-connect marks 28 -> 25
Other:
- moved on the sheet: J9
Changed lines of the file:
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@@
 	)
 	(no_connect
-		(at 130.81 144.78)
-	)
-	(no_connect
 		(at 77.47 130.81)
 	)
@@
 	)
 	(no_connect
-		(at 102.87 132.08)
-	)
-	(no_connect
 		(at 149.86 77.47)
 	)
@@
 	)
 	(no_connect
-		(at 130.81 129.54)
-	)
-	(no_connect
 		(at 113.03 40.64)
 	)
@@
 		)
 	)
-	(global_label "I00"
+	(global_label "IO0"
 		(shape output)
 		(at 269.24 161.29 0)
@@
 		)
 		(property "Intersheetrefs" "${INTERSHEET_REFS}"
-			(at 275.249 161.29 0)
+			(at 275.37 161.29 0)
 			(effects
 				(font
@@
 	(symbol
 		(lib_id "Connector_Generic:Conn_01x02")
-		(at 97.79 142.24 0)
-		(mirror y)
+		(at 97.79 144.78 180)
 		(unit 1)
 		(exclude_from_sim no)
@@
 		(dnp no)
 		(property "Reference" "J9"
-			(at 95.25 142.2399 0)
+			(at 95.504 142.748 0)
 			(effects
 				(font
@@
 		)
 		(property "Value" "Motor B"
-			(at 95.25 144.7799 0)
+			(at 95.504 144.526 0)
 			(effects
 				(font
@@
 			)
 		)
-		(property "Footprint" "Connector_JST:JST_XH_B2B-XH-AM_1x02_P2.50mm_Vertical"
-			(at 97.79 142.24 0)
+		(property "Footprint" "Connector_JST:JST_XH_B2B-XH-A_1x02_P2.50mm_Vertical"
+			(at 97.79 144.78 0)
 			(effects
 				(font
@@
 		)
 		(property "Datasheet" "~"
-			(at 97.79 142.24 0)
+			(at 97.79 144.78 0)
 			(effects
 				(font
@@
 		)
 		(property "Description" "Generic connector, single row, 01x02, script generated (kicad-library-utils/schlib/autogen/connector/)"
-			(at 97.79 142.24 0)
+			(at 97.79 144.78 0)
 			(effects
 				(font
@@
 			)
 		)
-		(property "Footprint" "esp32_devkit_v1_doit:H_Bridge"
+		(property "Footprint" "esp32_devkit_v1_doit:H_Bridge_with_headers"
 			(at 116.6368 135.6868 0)
 			(effects
@@
 					(size 1.27 1.27)
 				)
+				(hide yes)
 			)
 		)
@@
 		(on_board yes)
 		(dnp no)
-		(fields_autoplaced yes)
 		(property "Reference" "R3"
-			(at 57.15 173.9899 0)
+			(at 50.038 173.482 0)
 			(effects
 				(font
@@
 			)
 		)
-		(property "Value" "1K"
-			(at 57.15 176.5299 0)
+		(property "Value" "500R"
+			(at 48.006 176.276 0)
 			(effects
 				(font
@@
 			)
 		)
-		(property "Footprint" "Connector_JST:JST_XH_B5B-XH-AM_1x05_P2.50mm_Vertical"
+		(property "Footprint" "Connector_JST:JST_XH_B5B-XH-A_1x05_P2.50mm_Vertical"
 			(at 266.7 73.66 0)
 			(effects
@@
 		(dnp no)
 		(property "Reference" "D3"
-			(at 181.356 88.646 0)
+			(at 180.34 88.9 90)
 			(effects
 				(font
@@
 			)
 		)
-		(property "Value" "LED"
-			(at 180.34 91.7575 0)
+		(property "Value" "RED"
+			(at 180.34 91.44 90)
 			(effects
 				(font
@@
 		(on_board yes)
 		(dnp no)
-		(fields_autoplaced yes)
 		(property "Reference" "D1"
-			(at 58.42 184.4674 90)
+			(at 49.276 182.88 90)
 			(effects
 				(font
@@
 			)
 		)
-		(property "Value" "LED"
-			(at 58.42 187.0074 90)
+		(property "Value" "BLUE"
+			(at 48.26 185.166 90)
 			(effects
 				(font
@@
 		(on_board yes)
 		(dnp no)
-		(fields_autoplaced yes)
 		(property "Reference" "D5"
-			(at 119.38 183.1974 90)
+			(at 118.364 181.864 90)
 			(effects
 				(font
@@
 			)
 		)
-		(property "Value" "LED"
-			(at 119.38 185.7374 90)
+		(property "Value" "RED"
+			(at 118.364 184.15 90)
 			(effects
 				(font
@@
 			)
 		)
-		(property "Footprint" "Connector_JST:JST_XH_B2B-XH-AM_1x02_P2.50mm_Vertical"
+		(property "Footprint" "Connector_JST:JST_XH_B2B-XH-A_1x02_P2.50mm_Vertical"
 			(at 97.79 137.16 0)
 			(effects
@@
 		(dnp no)
 		(property "Reference" "R8"
-			(at 179.07 82.804 90)
+			(at 180.594 80.264 0)
 			(effects
 				(font
@@
 		)
 		(property "Value" "330"
-			(at 169.672 84.328 90)
+			(at 181.864 82.55 0)
 			(effects
 				(font
@@
 			)
 		)
-		(property "Footprint" "Connector_JST:JST_XH_B5B-XH-AM_1x05_P2.50mm_Vertical"
+		(property "Footprint" "Connector_JST:JST_XH_B5B-XH-A_1x05_P2.50mm_Vertical"
 			(at 266.7 43.18 0)
 			(effects
@@
 			)
 		)
-		(property "Footprint" "Connector_JST:JST_XH_B5B-XH-AM_1x05_P2.50mm_Vertical"
+		(property "Footprint" "Connector_JST:JST_XH_B5B-XH-A_1x05_P2.50mm_Vertical"
 			(at 266.7 59.69 0)
 			(effects
@@
 			)
 		)
-		(property "Footprint" "Button_Switch_THT:Nidec_Copal_SH-7010C"
+		(property "Footprint" "esp32_devkit_v1_doit:Push_Button_6_pins"
 			(at 42.164 170.434 0)
 			(effects
@@
 			)
 		)
-		(property "Value" "1K"
+		(property "Value" "130R"
 			(at 118.11 175.2599 0)
 			(effects
