File: Electronic_Modular/Sumo_Geral_Modular/Sumo_Geral_Modular.kicad_pcb (KiCad board)
At the start: 2 copper layers, 43.3 x 62.9 mm, 50 parts, among them J1 Bateria, J10 ESC1, J11 ESC2, J12 USB_B_Micro, J13 ADSN-9500, J14 ADSN-9500-PS, J15 MPU-6050, J2 VL53L0X 1, J3 VL53L0X 2, J4 VL53L0X 3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

Commit message: chore: update PCB and schematic
Parts:
- added C10: 100nF, Capacitor_SMD:C_0603_1608Metric, F.Cu at (158.7, 60.6)
- added C9: 100nF, Capacitor_SMD:C_0603_1608Metric, F.Cu at (160.2, 60.6)
- added J6: EXT2, Connector_PinHeader_2.00mm:PinHeader_1x03_P2.00mm_Vertical, F.Cu at (148.7, 64.3)
- added J7: EXT1, Connector_PinHeader_2.00mm:PinHeader_1x03_P2.00mm_Vertical, F.Cu at (148.7, 68.8)
- C7: value 100uF -> 100nF
- moved J12 5.50 mm to (149.8, 76.0)
- moved R11 4.37 mm to (160.2, 72.2), turned to 90 degrees
- moved R12 2.71 mm to (158.6, 72.2)
- moved J5 2.63 mm to (148.7, 60.1), turned to 90 degrees
- moved R14 2.58 mm to (158.7, 63.7), turned to -90 degrees
- moved D2 2.51 mm to (153.3, 78.9)
- moved R10 2.36 mm to (159.4, 69.8), turned to 180 degrees
- moved C8 1.51 mm to (160.2, 63.7)
- moved J15 0.82 mm to (156.1, 60.4)
Connections:
- ESP1 pad 10: AIN1 -> AIN2
- ESP1 pad 11: BIN1 -> AIN1
- ESP1 pad 12: ESC 1 -> BIN2/ESC2
- ESP1 pad 13: ESC 2 -> BIN1/ESC1
- ESP1 pad 14: BIN2 -> unconnected-(ESP1-IO12-Pad14)
- ESP1 pad 15: unconnected-(ESP1-GND-Pad15) -> GND
- ESP1 pad 16: AIN2 -> MOTION
- ESP1 pad 23: MOTION -> unconnected-(ESP1-IO15-Pad23)
- ESP1 pad 39: (no net) -> GND
- ESP1 pad 6: DDT -> IO34
- ESP1 pad 7: INT -> IO35
- ESP1 pad 8: unconnected-(ESP1-IO32-Pad8) -> INT
- ESP1 pad 9: unconnected-(ESP1-IO33-Pad9) -> DDT
- H_Bridge1 pad 11: BIN2 -> BIN2/ESC2
- H_Bridge1 pad 12: BIN1 -> BIN1/ESC1
- J10 pad 1: ESC 1 -> BIN1/ESC1
- J11 pad 1: ESC 2 -> BIN2/ESC2
Routing:
- net BIN2/ESC2: track 0.00 -> 32.1 mm
- net BIN1: track 24.3 -> 0.00 mm
- net ESC 2: track 24.2 -> 0.00 mm
- net BIN2: track 22.8 -> 0.00 mm
- net BIN1/ESC1: track 0.00 -> 22.8 mm
- net IO35: track 0.00 -> 14.1 mm
- net IO34: track 0.00 -> 12.7 mm
- net ESC 1: track 11.7 -> 0.00 mm
- net AIN2: track 9.58 -> 18.7 mm
- net MOTION: track 38.0 -> 29.2 mm
- net Net-(J12-D+): track 9.05 -> 15.8 mm
- net GND: track 0.00 -> 6.62 mm, vias 34 -> 38
- net Net-(D2-A): track 5.63 -> 0.00 mm
- net 3V3: track 209.4 -> 215.0 mm
- net SCL: track 101.7 -> 96.4 mm, vias 0 -> 1
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- added copper zone on B.Cu, net Net-(D2-A)
Other:
- board text added: "-"
- board text added: "34"
- board text added: "35"
- board text added: "BATT"
- board text added: "IR"
