File: Electronic_Modular/Sumo_Geral_Modular/Sumo_Geral_Modular.kicad_pcb (KiCad board)
At the start: 2 copper layers, 43.3 x 62.9 mm, 54 parts, among them J1 Bateria, J10 ESC1, J11 ESC2, J12 USB_B_Micro, J13 ADSN-9500, J14 ADSN-9500-PS, J15 MPU-6050, J2 VL53L0X 1, J3 VL53L0X 2, J4 VL53L0X 3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

Commit message: chore: update resistors values
Parts:
- R13: value 130R -> 75R/50mW
- R3: value 500R -> 300R/200mW
Changed lines of the file:
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@@
 			)
 		)
-		(property "Value" "500R"
+		(property "Value" "300R/200mW"
 			(at 0 1.43 90)
 			(layer "F.Fab")
@@
 		(tags "capacitor")
 		(property "Reference" "R10"
-			(at -0.015 1.45 360)
+			(at -0.015 1.45 0)
 			(layer "F.SilkS")
 			(effects
@@
 		)
 		(property "Value" "10K"
-			(at 0 1.43 360)
+			(at 0 1.43 0)
 			(layer "F.Fab")
 			(effects
@@
 		)
 		(fp_text user "${REFERENCE}"
-			(at 0 0 360)
+			(at 0 0 0)
 			(layer "F.Fab")
 			(effects
@@
 		)
 		(fp_text user "${REFERENCE}"
-			(at 0 2 360)
+			(at 0 2 0)
 			(layer "F.Fab")
 			(effects
@@
 			)
 		)
-		(property "Value" "130R"
+		(property "Value" "75R/50mW"
 			(at 0 1.43 90)
 			(layer "F.Fab")
@@
 		)
 		(fp_text user "${REFERENCE}"
-			(at 0 2 360)
+			(at 0 2 0)
 			(layer "F.Fab")
 			(effects
@@
 		)
 		(fp_text user "${REFERENCE}"
-			(at 0 2 360)
+			(at 0 2 0)
 			(layer "F.Fab")
 			(effects

Commit message: chore: create GERBER file
Other:
- board text added: "JLCJLCJLCJLC"
Changed lines of the file:
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@@
 			(outputformat 1)
 			(mirror no)
-			(drillshape 1)
+			(drillshape 0)
 			(scaleselection 1)
-			(outputdirectory "")
+			(outputdirectory "GERBER/")
 		)
 	)
@@
 		)
 	)
+	(gr_text "JLCJLCJLCJLC"
+		(at 170.9 55.43 0)
+		(layer "F.SilkS")
+		(effects
+			(font
+				(size 1 1)
+				(thickness 0.15)
+			)
+		)
+	)
